File: OpenJBOD-RP2040.kicad_pcb (KiCad board)
At the start: 4 copper layers, 72.6 x 170 mm, 122 parts, among them J1 ATX-24, J2 Bus_PCI_Express_x1, J3 Conn_02x02_Counter_Clockwise, J4 UART, J6 HR911105A, J8 USB_B_Micro, J9 TEMP1, Q1 MMBT3904, Q2 MMBT3904, SW1 SW_Push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

Commit message: rev4 order version added side-mounted IO to the panel so an IO shield could theoretically be made added step models cleaned up footprints
Parts:
- removed the D2 at (87.4, 133.5)
- removed the REF** at (96.8, 172.9) (x2)
- added REF**: OSHW-Logo2_9.8x8mm_SilkScreen, Symbol:OSHW-Logo2_9.8x8mm_SilkScreen, F.Cu at (94.8, 172.4)
- added REF**: OSHW-Logo2_9.8x8mm_SilkScreen, Symbol:OSHW-Logo2_9.8x8mm_SilkScreen, B.Cu at (94.8, 172.4)
- added SW3: TC-6615-6-260G, OpenJBOD_Library:KEY-TH_TC-6615-6-160G, F.Cu at (89.2, 126.8)
- D1: value GREEN -> MHK2396YGBTD; footprint LED_SMD:LED_0805_2012Metric -> OpenJBOD_Library:LED-TH_MHK2396YGBTD
- J4: footprint Connector_PinHeader_2.54mm:PinHeader_1x03_P2.54mm_Vertical -> Connector_PinHeader_2.54mm:PinHeader_1x03_P2.54mm_Horizontal
- SW2: value SW_Push -> TC-6615-6-260G; footprint Button_Switch_SMD:SW_Push_1P1T_XKB_TS-1187A -> OpenJBOD_Library:KEY-TH_TC-6615-6-160G
- moved SW1 15.2 mm to (101.8, 118.8), turned to 0 degrees
- moved J4 8.43 mm to (95.2, 98.6), turned to 180 degrees
- moved R1 5.52 mm to (95.1, 135.2), turned to -90 degrees
- moved R2 5.51 mm to (95.1, 133.2)
- moved Q2 5.33 mm to (99.4, 133.9)
- moved R27 5.33 mm to (101.9, 134.7)
- moved D1 4.53 mm to (91.8, 134.5), turned to -90 degrees
- moved SW2 1.17 mm to (89.2, 117.2), turned to -90 degrees
- renumbered D3 to D2, D4 to D3
Connections:
- net /SPI0_CSN renamed /SPI0_CSn
- net Net-(Q2-E) renamed /PICO_LED
- D1 pad 1: GND -> Net-(D1-Y_A)
- D1 pad 2: Net-(D1-A) -> GND
- J4 pad 1: /UART_TX -> /UART_RX
- J4 pad 2: /UART_RX -> /UART_TX
- R1 pad 1: Net-(D1-A) -> Net-(D1-G_A)
- R2 pad 1: Net-(D2-A) -> Net-(D1-Y_A)
Routing:
- net /PWR_BTN: track 38.6 -> 74.6 mm, vias 0 -> 1
- net /UART_RX: track 46.3 -> 38.7 mm
- net /UART_TX: track 49.0 -> 42.5 mm
- net /+3.3v: track 187.9 -> 182.6 mm
- net Net-(D1-G_A): track 0.00 -> 5.21 mm
- net /PICO_PWR: track 29.8 -> 24.9 mm
- net /+3.3vSB: track 223.5 -> 219.7 mm
- net /RUN: track 38.9 -> 35.2 mm, vias 2 -> 1
- net Net-(D1-Y_A): track 0.00 -> 2.26 mm
- net Net-(D2-A): track 1.48 -> 0.00 mm
- net Net-(D1-A): track 1.48 -> 0.00 mm
- net Net-(R8-Pad2): track 25.0 -> 26.0 mm
- net /PICO_LED: track 5.91 -> 5.40 mm
- net GND: vias 55 -> 56
Other:
- board text added: "POWER"
- board text removed: "JLCJLCJLCJLC"
- board text removed: "Rev4 production sponsored by:"
- board text removed: "Riff.CC"
