File: FanController.kicad_sch (KiCad schematic)
At the start: 13 parts, among them U6 EMC2301

Commit message: rev4.2
Updated silkscreen info block
Changed microUSB header to MicroXNJ
Added RoHS and WEEE marking
Moved BOOTSEL to rear IO
Moved SR latch
Moved J3 and J9 closer to the board edge, this helps to not interrupt
the 12v plane on inner layer 2
Parts:
- C33, C34, C35, C36, C37: JLCPCB_PN C110229 -> C2836440
Changed lines of the file:
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@@
 			)
 		)
-		(property "JLCPCB_PN" "C110229"
+		(property "JLCPCB_PN" "C2836440"
 			(at 140.97 80.01 0)
 			(effects
@@
 			)
 		)
-		(property "JLCPCB_PN" "C110229"
+		(property "JLCPCB_PN" "C2836440"
 			(at 140.97 60.96 0)
 			(effects
@@
 			)
 		)
-		(property "JLCPCB_PN" "C110229"
+		(property "JLCPCB_PN" "C2836440"
 			(at 140.97 118.11 0)
 			(effects
@@
 			)
 		)
-		(property "JLCPCB_PN" "C110229"
+		(property "JLCPCB_PN" "C2836440"
 			(at 140.97 43.18 0)
 			(effects
@@
 			)
 		)
-		(property "JLCPCB_PN" "C110229"
+		(property "JLCPCB_PN" "C2836440"
 			(at 140.97 99.06 0)
 			(effects
