File: MCU.kicad_sch (KiCad schematic)
At the start: 25 parts, among them SW1 TC-6615-6-260G, SW2 TC-6615-6-260G, U1 RP2040, U3 W25Q128JVS, Y1 X322512MSB4SI

Commit message: rev5
Added MACROM (specific ROM holding MAC address and (optionally) board
revision)
Added more circuitry to protect the EMC2301, allowing for use with fans
with internal pull-ups.
Added USB-C
Parts:
- added J8: TC2030-IDC-NL, Connector:Tag-Connect_TC2030-IDC-NL_2x03_P1.27mm_Vertical, symbol OpenJBOD:TC2030
- added TP1, TP2: TestPoint, TestPoint:TestPoint_Pad_D1.0mm, symbol Connector:TestPoint
- added U9: 24AA025E-OT, Package_TO_SOT_SMD:SOT-23-6, symbol Memory_EEPROM:24AA025E-OT
- C10, C11, C12, C13, C14, C4, C5, C7, C8, C9: JLCPCB_PN C1525 -> (none); LCSC Part # (none) -> C1525
- C15, C16: JLCPCB_PN C1658 -> (none); LCSC Part # (none) -> C1658
- C3, C6: JLCPCB_PN C52923 -> (none); LCSC Part # (none) -> C52923
- R18, R30: JLCPCB_PN C25900 -> (none); LCSC Part # (none) -> C25900
- R3, R4: value 27.4 -> 27.4R; JLCPCB_PN C284479 -> (none); LCSC Part # (none) -> C284479
- R8, R9: JLCPCB_PN C11702 -> (none); LCSC Part # (none) -> C11702
- SW1, SW2: JLCPCB_PN C2845272 -> (none); LCSC Part # (none) -> C2845272
- U1: JLCPCB_PN C2040 -> (none); LCSC Part # (none) -> C2040
- U3: JLCPCB_PN C97521 -> (none); LCSC Part # (none) -> C97521
- Y1: JLCPCB_PN C9002 -> (none); LCSC Part # (none) -> C9002
Connections:
- net +3.3vSB: now also J8.1, U9.6 (V_{CC})
- net GND: now also J8.6, U9.2 (V_{SS}), U9.4 (A1), U9.5 (A0)
- net RUN: now also TP1.1
- net USB_D+: now also J8.3
- net USB_D-: now also J8.5
- net at R8.2, SW1.2: now also TP2.1
- net FAN_SCL renamed I2C0_SCL
- net I2C0_SCL: now also J8.4, U9.1 (SCL)
- net FAN_SDA renamed I2C0_SDA
- net I2C0_SDA: now also J8.2, U9.3 (SDA)
Other:
- moved on the sheet: SW1, SW2
